File: BCoin2024.kicad_pcb (KiCad board)
At the start: 2 copper layers, 50 x 50 mm, 23 parts, among them U1 NE555DR, U2 74HC4017D_653

Commit message: Added PCBWAY PN text to rear of board, generated new gerbers for it
Other:
- board text added: "WayWayWay"
Changed lines of the file:
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@@
 		(layer "Edge.Cuts")
+	)
+	(gr_text "WayWayWay"
+		(at 134.75 105.75 0)
+		(layer "B.SilkS")
+		(effects
+			(font
+				(size 1 0.8)
+				(thickness 0.1)
+			)
+			(justify bottom mirror)
+		)
 	)
 	(gr_text "S+1\nVCC"
@@
 	)
 	(gr_text "2nd Thursday of the month\nPrime Time Restaurant\nHickory Hills\n95th St\n6:30 PM"
-		(at 134.5 107.5 0)
+		(at 134.5 101.75 0)
 		(layer "B.SilkS")
 		(effects
